Commit message: finished urdf file, fixed small bugs got differential_driver working

File: spooky/urdf/spooky_4wheel.urdf (robot description, URDF)
Before this commit: robot spooky, 6 links, 5 joints
Links:
- link base_laser: geometry visual cylinder length=0.0682625 radius=0.034925
- link base_link: geometry visual box size=.2905125 .1016 .034925
Joints:
- joint base_to_laser: origin xyz=-0.0889 0 0.0635 rpy=0 0 0 -> xyz=-0.0889 0 0.0587375 rpy=0 0 0
